File: electronica.kicad_sch (KiCad schematic)
At the start: 5 parts, among them U1 ESP32-DevKitC

Commit message: feat: integrated rtc ldc i2c / fixed 12v power line rs485 / output com pin -> input power type
Other:
- sheet power ports: added 12V; removed none
- sheet rs485 ports: added 12V; removed none
Changed lines of the file:
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@@
+	(wire
+		(pts
+			(xy 29.21 148.59) (xy 36.83 148.59)
+		)
+		(stroke
+			(width 0)
+			(type default)
+		)
+	)
 	(wire
 		(pts
@@
 		(pts
 			(xy 59.69 40.64) (xy 66.04 40.64)
+		)
+		(stroke
+			(width 0)
+			(type default)
+		)
+	)
+	(wire
+		(pts
+			(xy 33.02 49.53) (xy 36.83 49.53)
 		)
 		(stroke
@@
 		)
 	)
+	(label "12V"
+		(at 29.21 148.59 0)
+		(effects
+			(font
+				(size 1.27 1.27)
+			)
+			(justify left bottom)
+		)
+	)
 	(label "5V"
 		(at 29.21 74.93 0)
@@
 		(property "Intersheetrefs" "${INTERSHEET_REFS}"
 			(at 190.7805 146.05 0)
+			(effects
+				(font
+					(size 1.27 1.27)
+				)
+				(justify right)
+				(hide yes)
+			)
+		)
+	)
+	(global_label "12V"
+		(shape input)
+		(at 33.02 49.53 180)
+		(fields_autoplaced yes)
+		(effects
+			(font
+				(size 1.27 1.27)
+			)
+			(justify right)
+		)
+		(property "Intersheetrefs" "${INTERSHEET_REFS}"
+			(at 26.5272 49.53 0)
 			(effects
 				(font
@@
 			)
 		)
+		(pin "12V" input
+			(at 36.83 49.53 180)
+			(effects
+				(font
+					(size 1.27 1.27)
+				)
+				(justify left)
+			)
+		)
 		(instances
 			(project "electronica"
@@
 			(effects
 				(font
+					(size 1.27 1.27)
+				)
+				(justify left)
+			)
+		)
+		(pin "12V" input
+			(at 36.83 148.59 180)
+			(effects
+				(font
